File: Hardware/analog_outputs.kicad_sch (KiCad schematic)
At the start: 0 parts

Commit message: scheme update
Other:
- title: (none) -> PLC ON STM
Changed lines of the file:
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@@
 	(paper "A4")
 	(title_block
+		(title "PLC ON STM")
 		(company "Author: Grzegorz Potocki")
 	)

Commit message: schematic update
Parts:
- added C22, C23: 100n, Capacitor_SMD:C_0603_1608Metric_Pad1.08x0.95mm_HandSolder, symbol Device:C_Small
- added R22, R87: 33k, symbol Device:R_Small
- added R23, R88: 470R, symbol Device:R_Small
- added R24, R25: 1k, Resistor_SMD:R_0603_1608Metric_Pad0.98x0.95mm_HandSolder, symbol Device:R_Small
- added R26, R27: 100k, Resistor_SMD:R_0603_1608Metric_Pad0.98x0.95mm_HandSolder, symbol Device:R_Small
- added R85, R89: 10k, symbol Device:R_Small
- added R86, R90: 15k3, symbol Device:R_Small
- added U23, U24, U4: MCP6002-xSN, Package_SO:SOIC-8_3.9x4.9mm_P1.27mm, symbol Amplifier_Operational:MCP6002-xSN
- added U5: MCP6002-xSN, symbol Amplifier_Operational:MCP6002-xSN
Connections:
- new net: R22.2, R23.1, U23.2 (-)
- new net: R23.2, R85.2, R86.1
- new net: R22.1, U23.1
- new net: U23.3 (+), U4.1, U4.2 (-)
- new net: C23.1, R25.2, U5.3 (+)
- new net: C22.1, R24.2, U4.3 (+)
- new net: R88.2, R89.2, R90.1
- new net: R87.1, U24.1
- new net: R87.2, R88.1, U24.2 (-)
- new net: U24.3 (+), U5.1, U5.2 (-)
- new net +5V: R86.2, R90.2
- new net AO0: R24.1, R26.2
- new net AO1: R25.1, R27.2
- new net GND: C22.2, C23.2, R26.1, R27.1, R85.1, R89.1
Other:
- note added: "ANALOG OUTPUTS"
- note added: "OP AMPS POWER"
