File: Hardware/can.kicad_sch (KiCad schematic)
At the start: 14 parts, among them U2 ADM3057ExRW

Commit message: scheme update
Other:
- title: (none) -> PLC ON STM
Changed lines of the file:
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@@
 	(paper "A4")
 	(title_block
+		(title "PLC ON STM")
 		(company "Author: Grzegorz Potocki")
 	)

Commit message: schematic update
Parts:
- renumbered C15 to C32, C16 to C33, C17 to C34, C18 to C35, C19 to C36, C20 to C37, C21 to C38, C22 to C39, R7 to R84, U2 to U22
Changed lines of the file:
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@@
 		(on_board yes)
 		(dnp no)
-		(property "Reference" "R7"
+		(property "Reference" "R84"
 			(at 128.778 119.38 90)
 			(effects
@@
 			(project "stm32-plc"
 				(path "/b652b05a-4e3d-4ad1-b032-18886abe7d45/e88a87f1-4fac-4a15-8fc8-a85c85ae592e"
-					(reference "R7")
+					(reference "R84")
 					(unit 1)
 				)
@@
 		(dnp no)
 		(fields_autoplaced yes)
-		(property "Reference" "#PWR014"
+		(property "Reference" "#PWR043"
 			(at 184.15 119.38 0)
 			(effects
@@
 			(project "stm32-plc"
 				(path "/b652b05a-4e3d-4ad1-b032-18886abe7d45/e88a87f1-4fac-4a15-8fc8-a85c85ae592e"
-					(reference "#PWR014")
+					(reference "#PWR043")
 					(unit 1)
 				)
@@
 		(on_board yes)
 		(dnp no)
-		(property "Reference" "C18"
+		(property "Reference" "C35"
 			(at 124.46 113.03 0)
 			(effects
@@
 			(project "stm32-plc"
 				(path "/b652b05a-4e3d-4ad1-b032-18886abe7d45/e88a87f1-4fac-4a15-8fc8-a85c85ae592e"
-					(reference "C18")
+					(reference "C35")
 					(unit 1)
 				)
@@
 		(dnp no)
 		(fields_autoplaced yes)
-		(property "Reference" "#PWR015"
+		(property "Reference" "#PWR044"
 			(at 201.93 82.55 0)
 			(effects
@@
 			(project "stm32-plc"
 				(path "/b652b05a-4e3d-4ad1-b032-18886abe7d45/e88a87f1-4fac-4a15-8fc8-a85c85ae592e"
-					(reference "#PWR015")
+					(reference "#PWR044")
 					(unit 1)
 				)
@@
 		(on_board yes)
 		(dnp no)
-		(property "Reference" "C22"
+		(property "Reference" "C39"
 			(at 195.5863 80.01 90)
 			(effects
@@
 			(project "stm32-plc"
 				(path "/b652b05a-4e3d-4ad1-b032-18886abe7d45/e88a87f1-4fac-4a15-8fc8-a85c85ae592e"
-					(reference "C22")
+					(reference "C39")
 					(unit 1)
 				)
@@
 		(on_board yes)
 		(dnp no)
-		(property "Reference" "C17"
+		(property "Reference" "C34"
 			(at 105.41 113.03 0)
 			(effects
@@
 			(project "stm32-plc"
 				(path "/b652b05a-4e3d-4ad1-b032-18886abe7d45/e88a87f1-4fac-4a15-8fc8-a85c85ae592e"
-					(reference "C17")
+					(reference "C34")
 					(unit 1)
 				)
@@
 		(dnp no)
 		(fields_autoplaced yes)
-		(property "Reference" "#PWR011"
+		(property "Reference" "#PWR040"
 			(at 157.48 137.16 0)
 			(effects
@@
 			(project "stm32-plc"
 				(path "/b652b05a-4e3d-4ad1-b032-18886abe7d45/e88a87f1-4fac-4a15-8fc8-a85c85ae592e"
-					(reference "#PWR011")
+					(reference "#PWR040")
 					(unit 1)
 				)
@@
 		(on_board yes)
 		(dnp no)
-		(property "Reference" "C20"
+		(property "Reference" "C37"
 			(at 161.2837 80.01 90)
 			(effects
@@
 			(project "stm32-plc"
 				(path "/b652b05a-4e3d-4ad1-b032-18886abe7d45/e88a87f1-4fac-4a15-8fc8-a85c85ae592e"
-					(reference "C20")
+					(reference "C37")
 					(unit 1)
 				)
@@
 		(on_board yes)
 		(dnp no)
-		(property "Reference" "C15"
+		(property "Reference" "C32"
 			(at 91.44 125.73 0)
 			(effects
@@
 			(project "stm32-plc"
 				(path "/b652b05a-4e3d-4ad1-b032-18886abe7d45/e88a87f1-4fac-4a15-8fc8-a85c85ae592e"
-					(reference "C15")
+					(reference "C32")
 					(unit 1)
 				)
@@
 		(dnp no)
 		(fields_autoplaced yes)
-		(property "Reference" "#PWR013"
+		(property "Reference" "#PWR042"
 			(at 180.34 63.5 0)
 			(effects
@@
 			(project "stm32-plc"
 				(path "/b652b05a-4e3d-4ad1-b032-18886abe7d45/e88a87f1-4fac-4a15-8fc8-a85c85ae592e"
-					(reference "#PWR013")
+					(reference "#PWR042")
 					(unit 1)
 				)
@@
 		(dnp no)
 		(fields_autoplaced yes)
-		(property "Reference" "#PWR010"
+		(property "Reference" "#PWR039"
 			(at 154.94 82.55 0)
 			(effects
@@
 			(project "stm32-plc"
 				(path "/b652b05a-4e3d-4ad1-b032-18886abe7d45/e88a87f1-4fac-4a15-8fc8-a85c85ae592e"
-					(reference "#PWR010")
+					(reference "#PWR039")
 					(unit 1)
 				)
@@
 		(dnp no)
 		(fields_autoplaced yes)
-		(property "Reference" "C21"
+		(property "Reference" "C38"
 			(at 195.5863 55.88 90)
 			(effects
@@
 			(project "stm32-plc"
 				(path "/b652b05a-4e3d-4ad1-b032-18886abe7d45/e88a87f1-4fac-4a15-8fc8-a85c85ae592e"
-					(reference "C21")
+					(reference "C38")
 					(unit 1)
 				)
@@
 		(dnp no)
 		(fields_autoplaced yes)
-		(property "Reference" "#PWR012"
+		(property "Reference" "#PWR041"
 			(at 173.99 63.5 0)
 			(effects
@@
 			(project "stm32-plc"
 				(path "/b652b05a-4e3d-4ad1-b032-18886abe7d45/e88a87f1-4fac-4a15-8fc8-a85c85ae592e"
-					(reference "#PWR012")
+					(reference "#PWR041")
 					(unit 1)
 				)
@@
 		(on_board yes)
 		(dnp no)
-		(property "Reference" "U2"
+		(property "Reference" "U22"
 			(at 163.83 127 0)
 			(effects
@@
 			(project "stm32-plc"
 				(path "/b652b05a-4e3d-4ad1-b032-18886abe7d45/e88a87f1-4fac-4a15-8fc8-a85c85ae592e"
-					(reference "U2")
+					(reference "U22")
 					(unit 1)
 				)
@@
 		(on_board yes)
 		(dnp no)
-		(property "Reference" "C16"
+		(property "Reference" "C33"
 			(at 102.87 125.73 0)
 			(effects
@@
 			(project "stm32-plc"
 				(path "/b652b05a-4e3d-4ad1-b032-18886abe7d45/e88a87f1-4fac-4a15-8fc8-a85c85ae592e"
-					(reference "C16")
+					(reference "C33")
 					(unit 1)
 				)
@@
 		(on_board yes)
 		(dnp no)
-		(property "Reference" "C19"
+		(property "Reference" "C36"
 			(at 161.2963 55.88 90)
 			(effects
@@
 			(project "stm32-plc"
 				(path "/b652b05a-4e3d-4ad1-b032-18886abe7d45/e88a87f1-4fac-4a15-8fc8-a85c85ae592e"
-					(reference "C19")
-					(unit 1)
-				)
+					(reference "C36")
+					(unit 1)
+				)
