File: Hardware/connectors.kicad_sch (KiCad schematic)
At the start: 0 parts

Commit message: scheme update
Other:
- title: (none) -> PLC ON STM
Changed lines of the file:
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@@
 	(paper "A4")
 	(title_block
+		(title "PLC ON STM")
 		(company "Author: Grzegorz Potocki")
 	)

Commit message: schematic update
Parts:
- added D1, D2: SP0504BAJT, Package_TO_SOT_SMD:SOT-353_SC-70-5, symbol Power_Protection:SP0504BAJT
- added D3: PESD5V0L2BT,215, Package_TO_SOT_SMD:SOT-23-3, symbol Device:D_TVS_Dual_AAC
- added D4: SP0502BAHT, Package_TO_SOT_SMD:SOT-23, symbol Power_Protection:SP0502BAHT
- added J1: DIGITAL INPUT, symbol Connector:Screw_Terminal_01x08
- added J2: DIGITAL OUTPUT, symbol Connector:Screw_Terminal_01x08
- added J3: CAN, symbol Connector:Screw_Terminal_01x02
- added J4: POWER, symbol Connector:Screw_Terminal_01x02
- added J5: ANALOG INPUTS, symbol Connector:Screw_Terminal_01x02
- added J6: ANALOG OUTPUTS, symbol Connector:Screw_Terminal_01x02
- added J7: UART, symbol Connector:Screw_Terminal_01x04
Connections:
- new net +24V: J4.2 (Pin_2)
- new net +5V: J7.1 (Pin_1)
- new net ANALOG_IN0: J5.2 (Pin_2)
- new net ANALOG_IN1: J5.1 (Pin_1)
- new net ANALOG_OUT0: J6.2 (Pin_2)
- new net ANALOG_OUT1: J6.1 (Pin_1)
- new net CAN.N: D3.1 (A1), J3.2 (Pin_2)
- new net CAN.P: D3.2 (A2), J3.1 (Pin_1)
- new net CAN_GND_ISO: D3.3 (common)
- new net DI_IN0: D1.1 (K), J1.1 (Pin_1)
- new net DI_IN1: D1.3 (K), J1.2 (Pin_2)
- new net DI_IN2: D1.4 (K), J1.3 (Pin_3)
- new net DI_IN3: D1.5 (K), J1.4 (Pin_4)
- new net DI_IN4: D2.1 (K), J1.5 (Pin_5)
- new net DI_IN5: D2.3 (K), J1.6 (Pin_6)
- new net DI_IN6: D2.4 (K), J1.7 (Pin_7)
- new net DI_IN7: D2.5 (K), J1.8 (Pin_8)
- new net DI_OUT0: J2.1 (Pin_1)
- new net DI_OUT1: J2.2 (Pin_2)
- new net DI_OUT2: J2.3 (Pin_3)
- new net DI_OUT3: J2.4 (Pin_4)
- new net DI_OUT4: J2.5 (Pin_5)
- new net DI_OUT5: J2.6 (Pin_6)
- new net DI_OUT6: J2.7 (Pin_7)
- new net DI_OUT7: J2.8 (Pin_8)
- new net GND: D1.2 (A), D2.2 (A), D4.3 (A), J7.4 (Pin_4)
- new net GNDREF: J4.1 (Pin_1)
- new net UART.RX: D4.2 (K), J7.3 (Pin_3)
- new net UART.TX: D4.1 (K), J7.2 (Pin_2)
Other:
- note added: "ANALOG INPUT CONNECTOR"
- note added: "ANALOG OUTPUT CONNECTOR"
- note added: "CAN CONNECTOR"
- note added: "DIGITAL INPUT CONNECTOR"
- note added: "DIGITAL OUTPUT CONNECTOR"
- note added: "ESD ANALOG PROTECTION"
- note added: "ESD CAN PROTECTION"
- note added: "ESD DIGITAL PROTECTION"
- note added: "ESD UART PROTECTION"
- note added: "POWER CONNECTOR"
- note added: "UART CONNECTOR"
