File: Hardware/digital_outputs.kicad_sch (KiCad schematic)
At the start: 0 parts

Commit message: scheme update
Other:
- title: (none) -> PLC ON STM
Changed lines of the file:
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@@
 	(paper "A4")
 	(title_block
+		(title "PLC ON STM")
 		(company "Author: Grzegorz Potocki")
 	)

Commit message: schematic update
Parts:
- added Q10, Q11, Q12, Q13, Q14, Q15, Q16, Q17: PMOS, symbol Simulation_SPICE:PMOS
- added R60, R61, R62, R63, R64, R65, R66, R67: 47k, symbol Device:R_Small
- added R68, R69, R70, R71, R72, R73, R74, R75, R76, R77, R78, R79, R80, R81, R82, R83: 1k, symbol Device:R_Small
- added U14, U15, U16, U17, U18, U19, U20, U21: CNY17-4, symbol Isolator:CNY17-4
Connections:
- new net: R72.1, U18.1
- new net: Q14.1 (D), U18.2
- new net: Q13.1 (D), U17.2
- new net: Q13.2 (G), R79.1
- new net: R68.1, U14.1
- new net: Q10.1 (D), U14.2
- new net: Q16.1 (D), U20.2
- new net: Q16.2 (G), R82.1
- new net: Q11.1 (D), U15.2
- new net: Q11.2 (G), R77.1
- new net: Q12.2 (G), R78.1
- new net: R69.1, U15.1
- new net: R71.1, U17.1
- new net: R75.1, U21.1
- new net: Q10.2 (G), R76.1
- new net: Q17.1 (D), U21.2
- new net: R74.1, U20.1
- new net: R73.1, U19.1
- new net: Q15.1 (D), U19.2
- new net: Q15.2 (G), R81.1
- new net: R70.1, U16.1
- new net: Q14.2 (G), R80.1
- new net: Q12.1 (D), U16.2
- new net: Q17.2 (G), R83.1
- new net +24V: U14.5, U15.5, U16.5, U17.5, U18.5, U19.5, U20.5, U21.5
- new net +5V: R68.2, R69.2, R70.2, R71.2, R72.2, R73.2, R74.2, R75.2
- new net DI_OUT0: R60.1, U14.4
- new net DI_OUT1: R61.1, U15.4
- new net DI_OUT2: R62.1, U16.4
- new net DI_OUT3: R63.1, U17.4
- new net DI_OUT4: R64.1, U18.4
- new net DI_OUT5: R65.1, U19.4
- new net DI_OUT6: R66.1, U20.4
- new net DI_OUT7: R67.1, U21.4
- new net DO0: R76.2
- new net DO1: R77.2
- new net DO2: R78.2
- new net DO3: R79.2
- new net DO4: R80.2
- new net DO5: R81.2
- new net DO6: R82.2
- new net DO7: R83.2
- new net GND: Q10.3 (S), Q11.3 (S), Q12.3 (S), Q13.3 (S), Q14.3 (S), Q15.3 (S), Q16.3 (S), Q17.3 (S)
- new net GNDREF: R60.2, R61.2, R62.2, R63.2, R64.2, R65.2, R66.2, R67.2
- no-connect marks 0 -> 8
Other:
- note added: "DIGITAL OUTPUTS"
- note added: "Galvanic isolation"
