File: Hardware/uart.kicad_sch (KiCad schematic)
At the start: 0 parts

Commit message: scheme update
Other:
- title: (none) -> PLC ON STM
Changed lines of the file:
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@@
 	(paper "A4")
 	(title_block
+		(title "PLC ON STM")
 		(company "Author: Grzegorz Potocki")
 	)

Commit message: schematic update
Parts:
- added C40, C41: 1u, symbol Device:C_Small
- added IC1: ISO7721FQDWVRQ1, SOIC127P1150X280-8N, symbol PLC_on_STM:ISO7721FQDWVRQ1
Connections:
- new net +3V3: C40.1, C41.1, IC1.1 (VCC1), IC1.8 (VCC2)
- new net GNDREF: C40.2, C41.2, IC1.4 (GND1), IC1.5 (GND2)
- new net UART.RX: IC1.2 (OUTA)
- new net UART.TX: IC1.3 (INB)
- new net UART_ISO.RX: IC1.6 (OUTB)
- new net UART_ISO.TX: IC1.7 (INA)
Other:
- note added: "Isolation"
- note added: "UART ISOLATION"
