File: Hardware/DigitalOutput/digitalIO.kicad_pcb (KiCad board)
At the start: 4 copper layers, 70 x 66.8 mm, 140 parts, among them J1 DIGITAL INPUT, J2 DIGITAL OUTPUT, J3 Conn_02x23_Odd_Even, J4 Conn_02x23_Odd_Even, Q1 SI2347DS, Q10 SI2347DS, Q11 SI2347DS, Q12 SI2347DS, Q13 SI2347DS, Q14 SI2347DS, Q15 SI2347DS, Q16 SI2347DS, Q2 SI2347DS, Q3 SI2347DS, Q4 SI2347DS, Q5 SI2347DS, Q6 SI2347DS, Q7 SI2347DS, Q8 SI2347DS, Q9 SI2347DS, U1 CNY17-3, U10 CNY17-3, U11 CNY17-3, U12 CNY17-3, U13 CNY17-3, U14 CNY17-3, U15 CNY17-3, U16 CNY17-3, U2 CNY17-3, U3 CNY17-3, U4 CNY17-3, U5 CNY17-3, U6 CNY17-3, U7 CNY17-3, U8 CNY17-3, U9 CNY17-3

Commit message: schematic update & pcb update
Parts:
- moved J3 0.08 mm to (182.8, 108.5)
- moved J4 0.08 mm to (119.2, 52.5)
Other:
- board size 70 x 66.8 mm -> 70 x 64.8 mm
Changed lines of the file:
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@@
 	(footprint "PLC_STM:PRT12790"
 		(layer "F.Cu")
-		(at 119.25 52.45 -90)
+		(at 119.25 52.535 -90)
 		(descr "PRT-12790-1")
 		(tags "Connector")
@@
 	(footprint "PLC_STM:PRT12790"
 		(layer "F.Cu")
-		(at 182.75 108.4 90)
+		(at 182.75 108.485 90)
 		(descr "PRT-12790-1")
 		(tags "Connector")
@@
 	)
 	(gr_arc
-		(start 137 57.085)
-		(mid 136.292893 56.792107)
-		(end 136 56.085)
+		(start 137 57.17)
+		(mid 136.292893 56.877107)
+		(end 136 56.17)
 		(stroke
 			(width 0.15)
@@
 	)
 	(gr_line
-		(start 127 113.915)
-		(end 129 115.915)
+		(start 162 100)
+		(end 129 100)
+		(stroke
+			(width 0.15)
+			(type solid)
+		)
+		(layer "Edge.Cuts")
+	)
+	(gr_line
+		(start 164 114)
+		(end 164 102)
 		(stroke
 			(width 0.15)
@@
 	)
 	(gr_arc
-		(start 185 49.085)
-		(mid 185.707107 49.377893)
-		(end 186 50.085)
+		(start 185 49.17)
+		(mid 185.707107 49.462893)
+		(end 186 50.17)
 		(stroke
 			(width 0.15)
@@
 	)
 	(gr_arc
-		(start 166 50.085)
-		(mid 166.292893 49.377893)
-		(end 167 49.085)
+		(start 166 50.17)
+		(mid 166.292893 49.462893)
+		(end 167 49.17)
 		(stroke
 			(width 0.15)
@@
 	)
 	(gr_line
-		(start 164 113.915)
-		(end 184 113.915)
+		(start 164 114)
+		(end 184 114)
 		(stroke
 			(width 0.15)
@@
 	)
 	(gr_arc
-		(start 186 111.915)
-		(mid 185.414214 113.329214)
-		(end 184 113.915)
+		(start 186 112)
+		(mid 185.414214 113.414214)
+		(end 184 114)
 		(stroke
 			(width 0.15)
@@
 	)
 	(gr_line
-		(start 166 50.085)
-		(end 166 56.085)
+		(start 166 50.17)
+		(end 166 56.17)
 		(stroke
 			(width 0.15)
@@
 	)
 	(gr_arc
-		(start 116 50.085)
-		(mid 116.292893 49.377893)
-		(end 117 49.085)
+		(start 116 50.17)
+		(mid 116.292893 49.462893)
+		(end 117 49.17)
 		(stroke
 			(width 0.15)
@@
 	)
 	(gr_circle
-		(center 126.87 53.505)
-		(end 128.49 53.505)
+		(center 126.87 53.59)
+		(end 128.49 53.59)
 		(stroke
 			(width 0.15)
@@
 		(layer "Edge.Cuts")
 	)
-	(gr_line
-		(start 162 115.915)
-		(end 164 113.915)
+	(gr_circle
+		(center 159.87 96.63)
+		(end 161.5 96.63)
 		(stroke
 			(width 0.15)
 			(type solid)
 		)
+		(fill no)
 		(layer "Edge.Cuts")
 	)
-	(gr_circle
-		(center 159.87 113.415)
-		(end 161.5 113.415)
+	(gr_line
+		(start 127 114)
+		(end 127 102)
 		(stroke
 			(width 0.15)
 			(type solid)
 		)
-		(fill no)
 		(layer "Edge.Cuts")
 	)
 	(gr_line
-		(start 118 113.915)
-		(end 127 113.915)
+		(start 118 114)
+		(end 127 114)
 		(stroke
 			(width 0.15)
@@
 	)
 	(gr_circle
-		(center 175.13 54.785)
-		(end 176.75 54.785)
+		(center 175.13 54.87)
+		(end 176.75 54.87)
 		(stroke
 			(width 0.15)
@@
 	)
 	(gr_arc
-		(start 135 49.085)
-		(mid 135.707107 49.377893)
-		(end 136 50.085)
+		(start 135 49.17)
+		(mid 135.707107 49.462893)
+		(end 136 50.17)
 		(stroke
 			(width 0.15)
@@
 	)
 	(gr_arc
-		(start 118 113.915)
-		(mid 116.585786 113.329214)
-		(end 116 111.915)
+		(start 118 114)
+		(mid 116.585786 113.414214)
+		(end 116 112)
+		(stroke
+			(width 0.15)
+			(type solid)
+		)
+		(layer "Edge.Cuts")
+	)
+	(gr_line
+		(start 186 112)
+		(end 186 50.17)
 		(stroke
 			(width 0.15)
@@
 	)
 	(gr_line
-		(start 186 111.915)
-		(end 186 50.085)
+		(start 162 100)
+		(end 164 102)
 		(stroke
 			(width 0.15)
@@
 	)
 	(gr_line
-		(start 129 115.915)
-		(end 162 115.915)
+		(start 127 102)
+		(end 129 100)
 		(stroke
 			(width 0.15)
@@
 	)
 	(gr_line
-		(start 185 49.085)
-		(end 167 49.085)
+		(start 185 49.17)
+		(end 167 49.17)
 		(stroke
 			(width 0.15)
@@
 	)
 	(gr_arc
-		(start 166 56.085)
-		(mid 165.707107 56.792107)
-		(end 165 57.085)
+		(start 166 56.17)
+		(mid 165.707107 56.877107)
+		(end 165 57.17)
 		(stroke
 			(width 0.15)
@@
 	)
 	(gr_line
-		(start 117 49.085)
-		(end 135 49.085)
+		(start 117 49.17)
+		(end 135 49.17)
 		(stroke
 			(width 0.15)
@@
 	)
 	(gr_line
-		(start 165 57.085)
-		(end 137 57.085)
+		(start 165 57.17)
+		(end 137 57.17)
 		(stroke
 			(width 0.15)
@@
 	)
 	(gr_line
-		(start 136 50.085)
-		(end 136 56.085)
+		(start 136 50.17)
+		(end 136 56.17)
 		(stroke
 			(width 0.15)
@@
 	)
 	(gr_line
-		(start 116 111.915)
-		(end 116 50.085)
+		(start 116 112)
+		(end 116 50.17)
 		(stroke
 			(width 0.15)
@@
 	)
 	(gr_text "®©®"
-		(at 132.75 114.415 0)
+		(at 132.75 98 0)
 		(layer "B.Mask")
 		(effects
