File: Hardware/DigitalOutput/digital_output.kicad_pcb (KiCad board)
At the start: 4 copper layers, 70 x 59 mm, 2 parts, among them CN10 Conn_02x19_Odd_Even, CN7 Conn_02x19_Odd_Even

Commit message: digital output & power finished
Parts:
- removed CN10, CN7: Conn_02x19_Odd_Even, Connector_PinSocket_2.54mm:PinSocket_2x19_P2.54mm_Vertical
- added D1: LD_DO0, LED_SMD:LED_0603_1608Metric_Pad1.05x0.95mm_HandSolder, F.Cu at (127.5, 94.8)
- added D2: LD_DO1, LED_SMD:LED_0603_1608Metric_Pad1.05x0.95mm_HandSolder, F.Cu at (134.2, 94.8)
- added D3: LD_DO2, LED_SMD:LED_0603_1608Metric_Pad1.05x0.95mm_HandSolder, F.Cu at (140.5, 94.8)
- added D4: LD_DO3, LED_SMD:LED_0603_1608Metric_Pad1.05x0.95mm_HandSolder, F.Cu at (147.0, 94.8)
- added D5: LD_DO4, LED_SMD:LED_0603_1608Metric_Pad1.05x0.95mm_HandSolder, F.Cu at (154.0, 94.8)
- added D6: LD_DO5, LED_SMD:LED_0603_1608Metric_Pad1.05x0.95mm_HandSolder, F.Cu at (160.5, 94.8)
- added D7: LD_DO6, LED_SMD:LED_0603_1608Metric_Pad1.05x0.95mm_HandSolder, F.Cu at (167.0, 94.8)
- added D8: LD_DO7, LED_SMD:LED_0603_1608Metric_Pad1.05x0.95mm_HandSolder, F.Cu at (173.5, 94.8)
- added J1: DIGITAL OUTPUT, PLC_STM:1725724, F.Cu at (133.5, 111.0)
- added J2: NUCLEO LEFT, PLC_STM:PRT12790, F.Cu at (119.2, 52.5)
- added J3: NUCLEO RIGHT, PLC_STM:PRT12790, F.Cu at (180.2, 52.5)
- added Q1: SI2347DS, Package_TO_SOT_SMD:SOT-23-3, F.Cu at (129.2, 64.5)
- added Q2: SI2347DS, Package_TO_SOT_SMD:SOT-23-3, F.Cu at (135.5, 64.4)
- added Q3: SI2347DS, Package_TO_SOT_SMD:SOT-23-3, F.Cu at (141.8, 64.5)
- added Q4: SI2347DS, Package_TO_SOT_SMD:SOT-23-3, F.Cu at (148.0, 64.5)
- added Q5: SI2347DS, Package_TO_SOT_SMD:SOT-23-3, F.Cu at (155.0, 64.5)
- added Q6: SI2347DS, Package_TO_SOT_SMD:SOT-23-3, F.Cu at (161.2, 64.2)
- added Q7: SI2347DS, Package_TO_SOT_SMD:SOT-23-3, F.Cu at (167.5, 64.4)
- added Q8: SI2347DS, Package_TO_SOT_SMD:SOT-23-3, F.Cu at (173.8, 64.2)
- added R1: 47k, Resistor_SMD:R_0603_1608Metric_Pad0.98x0.95mm_HandSolder, F.Cu at (127.5, 91.8)
- added R10: 1k, Resistor_SMD:R_0603_1608Metric_Pad0.98x0.95mm_HandSolder, F.Cu at (135.8, 69.8)
- added R11: 1k, Resistor_SMD:R_0603_1608Metric_Pad0.98x0.95mm_HandSolder, F.Cu at (142.2, 69.8)
- added R12: 1k, Resistor_SMD:R_0603_1608Metric_Pad0.98x0.95mm_HandSolder, F.Cu at (148.8, 69.8)
- added R13: 1k, Resistor_SMD:R_0603_1608Metric_Pad0.98x0.95mm_HandSolder, F.Cu at (155.8, 69.8)
- added R14: 1k, Resistor_SMD:R_0603_1608Metric_Pad0.98x0.95mm_HandSolder, F.Cu at (162.2, 69.8)
- added R15: 1k, Resistor_SMD:R_0603_1608Metric_Pad0.98x0.95mm_HandSolder, F.Cu at (168.8, 69.8)
- added R16: 1k, Resistor_SMD:R_0603_1608Metric_Pad0.98x0.95mm_HandSolder, F.Cu at (175.2, 69.8)
- added R17: 1k, Resistor_SMD:R_0603_1608Metric_Pad0.98x0.95mm_HandSolder, F.Cu at (130.2, 60.5)
- added R18: 1k, Resistor_SMD:R_0603_1608Metric_Pad0.98x0.95mm_HandSolder, F.Cu at (136.5, 60.5)
- added R19: 1k, Resistor_SMD:R_0603_1608Metric_Pad0.98x0.95mm_HandSolder, F.Cu at (142.7, 60.5)
- added R2: 47k, Resistor_SMD:R_0603_1608Metric_Pad0.98x0.95mm_HandSolder, F.Cu at (134.2, 91.8)
- added R20: 1k, Resistor_SMD:R_0603_1608Metric_Pad0.98x0.95mm_HandSolder, F.Cu at (149.0, 60.5)
- added R21: 1k, Resistor_SMD:R_0603_1608Metric_Pad0.98x0.95mm_HandSolder, F.Cu at (156.0, 60.5)
- added R22: 1k, Resistor_SMD:R_0603_1608Metric_Pad0.98x0.95mm_HandSolder, F.Cu at (162.2, 60.5)
- added R23: 1k, Resistor_SMD:R_0603_1608Metric_Pad0.98x0.95mm_HandSolder, F.Cu at (168.5, 60.5)
- added R24: 1k, Resistor_SMD:R_0603_1608Metric_Pad0.98x0.95mm_HandSolder, F.Cu at (174.8, 60.5)
- added R3: 47k, Resistor_SMD:R_0603_1608Metric_Pad0.98x0.95mm_HandSolder, F.Cu at (140.5, 91.8)
- added R4: 47k, Resistor_SMD:R_0603_1608Metric_Pad0.98x0.95mm_HandSolder, F.Cu at (147.0, 91.8)
- added R5: 47k, Resistor_SMD:R_0603_1608Metric_Pad0.98x0.95mm_HandSolder, F.Cu at (154.0, 91.8)
- added R6: 47k, Resistor_SMD:R_0603_1608Metric_Pad0.98x0.95mm_HandSolder, F.Cu at (160.5, 91.8)
- added R7: 47k, Resistor_SMD:R_0603_1608Metric_Pad0.98x0.95mm_HandSolder, F.Cu at (167.0, 91.8)
- added R8: 47k, Resistor_SMD:R_0603_1608Metric_Pad0.98x0.95mm_HandSolder, F.Cu at (173.5, 91.8)
- added R9: 1k, Resistor_SMD:R_0603_1608Metric_Pad0.98x0.95mm_HandSolder, F.Cu at (129.2, 69.8)
- added U1: VO615A-3, Package_DIP:DIP-4_W8.89mm_SMDSocket_LongPads, F.Cu at (128.0, 78.2)
- added U2: VO615A-3, Package_DIP:DIP-4_W8.89mm_SMDSocket_LongPads, F.Cu at (134.5, 78.2)
- added U3: VO615A-3, Package_DIP:DIP-4_W8.89mm_SMDSocket_LongPads, F.Cu at (141.0, 78.2)
- added U4: VO615A-3, Package_DIP:DIP-4_W8.89mm_SMDSocket_LongPads, F.Cu at (147.5, 78.2)
- added U5: VO615A-3, Package_DIP:DIP-4_W8.89mm_SMDSocket_LongPads, F.Cu at (154.5, 78.2)
- added U6: VO615A-3, Package_DIP:DIP-4_W8.89mm_SMDSocket_LongPads, F.Cu at (161.0, 78.2)
- added U7: VO615A-3, Package_DIP:DIP-4_W8.89mm_SMDSocket_LongPads, F.Cu at (167.5, 78.2)
- added U8: VO615A-3, Package_DIP:DIP-4_W8.89mm_SMDSocket_LongPads, F.Cu at (174.0, 78.2)
Routing:
- net +5V: track 0.00 -> 107.4 mm, vias 0 -> 8
- net +24V: track 0.00 -> 88.4 mm, vias 0 -> 8
- net DO_3: track 0.00 -> 81.3 mm
- net DO_2: track 0.00 -> 71.5 mm
- net DO_4: track 0.00 -> 66.2 mm
- net DO_5: track 0.00 -> 56.5 mm
- net DO_1: track 0.00 -> 56.3 mm
- net DI_OUT7: track 0.00 -> 51.3 mm
- net DO_6: track 0.00 -> 50.4 mm
- net DI_OUT6: track 0.00 -> 46.7 mm
- net DO_0: track 0.00 -> 46.6 mm
- net DO_7: track 0.00 -> 45.6 mm
- net DI_OUT5: track 0.00 -> 42.8 mm
- net DI_OUT4: track 0.00 -> 39.7 mm
- net DI_OUT3: track 0.00 -> 37.8 mm
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- added copper zone on B.Cu, net GND
- added copper zone on F.Cu, net GND
- added copper zone on In1.Cu, net GND
- added copper zone on In2.Cu, net GND
- added copper zone on B.Cu, net GNDREF
- added copper zone on F.Cu, net GNDREF
- added copper zone on In1.Cu, net GNDREF
- added copper zone on In2.Cu, net GNDREF
Other:
- board size 70 x 59 mm -> 70 x 67.5 mm
- board text removed: "Template"
- board text removed: "v${REVISION}"
- board text removed: "®©®"

Commit message: small adjustments and final revision
Connections:
- J2 pad 36: DO_0 -> unconnected-(J2-Pin_36-Pad36)
- J2 pad 38: DO_1 -> unconnected-(J2-Pin_38-Pad38)
- J2 pad 40: DO_2 -> DO_0
- J2 pad 42: DO_3 -> DO_1
- J2 pad 44: unconnected-(J2-Pin_44-Pad44) -> DO_2
- J2 pad 46: unconnected-(J2-Pin_46-Pad46) -> DO_3
Routing:
- net DO_3: track 81.3 -> 86.6 mm
- net DO_1: track 56.3 -> 61.4 mm
- net DO_0: track 46.6 -> 51.7 mm
- net DO_2: track 71.5 -> 76.4 mm
Changed lines of the file:
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@@
 	(net 30 "unconnected-(J2-Pin_41-Pad41)")
 	(net 31 "unconnected-(J2-Pin_43-Pad43)")
-	(net 32 "unconnected-(J2-Pin_44-Pad44)")
+	(net 32 "unconnected-(J2-Pin_36-Pad36)")
 	(net 33 "unconnected-(J2-Pin_45-Pad45)")
-	(net 34 "unconnected-(J2-Pin_46-Pad46)")
+	(net 34 "unconnected-(J2-Pin_38-Pad38)")
 	(net 35 "unconnected-(J3-Pin_1-Pad1)")
 	(net 36 "unconnected-(J3-Pin_3-Pad3)")
@@
 			(layers "*.Cu" "*.Mask")
 			(remove_unused_layers no)
-			(net 88 "DO_0")
+			(net 32 "unconnected-(J2-Pin_36-Pad36)")
 			(pinfunction "Pin_36")
-			(pintype "passive")
+			(pintype "passive+no_connect")
 		)
 		(pad "37" thru_hole circle
@@
 			(layers "*.Cu" "*.Mask")
 			(remove_unused_layers no)
-			(net 96 "DO_1")
+			(net 34 "unconnected-(J2-Pin_38-Pad38)")
 			(pinfunction "Pin_38")
-			(pintype "passive")
+			(pintype "passive+no_connect")
 		)
 		(pad "39" thru_hole circle
@@
 			(layers "*.Cu" "*.Mask")
 			(remove_unused_layers no)
-			(net 95 "DO_2")
+			(net 88 "DO_0")
 			(pinfunction "Pin_40")
 			(pintype "passive")
@@
 			(layers "*.Cu" "*.Mask")
 			(remove_unused_layers no)
-			(net 91 "DO_3")
+			(net 96 "DO_1")
 			(pinfunction "Pin_42")
 			(pintype "passive")
@@
 			(layers "*.Cu" "*.Mask")
 			(remove_unused_layers no)
-			(net 32 "unconnected-(J2-Pin_44-Pad44)")
+			(net 95 "DO_2")
 			(pinfunction "Pin_44")
-			(pintype "passive+no_connect")
+			(pintype "passive")
 		)
 		(pad "45" thru_hole circle
@@
 			(layers "*.Cu" "*.Mask")
 			(remove_unused_layers no)
-			(net 34 "unconnected-(J2-Pin_46-Pad46)")
+			(net 91 "DO_3")
 			(pinfunction "Pin_46")
-			(pintype "passive+no_connect")
+			(pintype "passive")
 		)
 		(embedded_fonts no)
@@
 		(layer "Edge.Cuts")
 	)
+	(dimension
+		(type orthogonal)
+		(layer "Dwgs.User")
+		(pts
+			(xy 118 51.115) (xy 184 51.125)
+		)
+		(height -5.115)
+		(orientation 0)
+		(format
+			(prefix "")
+			(suffix "")
+			(units 3)
+			(units_format 1)
+			(precision 4)
+			(suppress_zeroes yes)
+		)
+		(style
+			(thickness 0.1)
+			(arrow_length 1.27)
+			(text_position_mode 1)
+			(arrow_direction outward)
+			(extension_height 0.58642)
+			(extension_offset 0.5)
+			(keep_text_aligned yes)
+		)
+		(gr_text "66 mm"
+			(at 151 46 0)
+			(layer "Dwgs.User")
+			(effects
+				(font
+					(size 0.8 0.8)
+					(thickness 0.1)
+				)
+			)
+		)
+	)
+	(dimension
+		(type orthogonal)
+		(layer "Dwgs.User")
+		(pts
+			(xy 116 112) (xy 186 112)
+		)
+		(height 14)
+		(orientation 0)
+		(format
+			(prefix "")
+			(suffix "")
+			(units 3)
+			(units_format 1)
+			(precision 4)
+			(suppress_zeroes yes)
+		)
+		(style
+			(thickness 0.1)
+			(arrow_length 1.27)
+			(text_position_mode 1)
+			(arrow_direction outward)
+			(extension_height 0.58642)
+			(extension_offset 0.5)
+			(keep_text_aligned yes)
+		)
+		(gr_text "70 mm"
+			(at 151 126 0)
+			(layer "Dwgs.User")
+			(effects
+				(font
+					(size 0.8 0.8)
+					(thickness 0.1)
+				)
+			)
+		)
+	)
+	(dimension
+		(type orthogonal)
+		(layer "Dwgs.User")
+		(pts
+			(xy 162 116) (xy 167 48.5)
+		)
+		(height 34)
+		(orientation 1)
+		(format
+			(prefix "")
+			(suffix "")
+			(units 3)
+			(units_format 1)
+			(precision 4)
+			(suppress_zeroes yes)
+		)
+		(style
+			(thickness 0.1)
+			(arrow_length 1.27)
+			(text_position_mode 1)
+			(arrow_direction outward)
+			(extension_height 0.58642)
+			(extension_offset 0.5)
+			(keep_text_aligned yes)
+		)
+		(gr_text "67.5 mm"
+			(at 196 82.25 90)
+			(layer "Dwgs.User")
+			(effects
+				(font
+					(size 0.8 0.8)
+					(thickness 0.1)
+				)
+			)
+		)
+	)
 	(segment
 		(start 173.75 64.3)
@@
 	)
 	(segment
-		(start 120.541 94.461)
-		(end 121.77 95.69)
+		(start 122.284536 61.377)
+		(end 121 61.377)
 		(width 0.2)
 		(layer "F.Cu")
@@
 	)
 	(segment
-		(start 120.541 61.836)
-		(end 120.541 94.461)
+		(start 120.541 99.541)
+		(end 121.77 100.77)
 		(width 0.2)
 		(layer "F.Cu")
@@
 	)
 	(segment
-		(start 121 61.377)
-		(end 120.541 61.836)
+		(start 120.541 61.836)
+		(end 120.541 99.541)
 		(width 0.2)
 		(layer "F.Cu")
@@
 	)
 	(segment
-		(start 122.284536 61.377)
-		(end 121 61.377)
+		(start 124.038536 59.623)
+		(end 122.284536 61.377)
 		(width 0.2)
 		(layer "F.Cu")
@@
 	)
 	(segment
-		(start 131.1625 60.5)
-		(end 131.1625 59.9125)
+		(start 131.1625 59.9125)
+		(end 130.873 59.623)
 		(width 0.2)
 		(layer "F.Cu")
@@
 	)
 	(segment
-		(start 131.1625 59.9125)
-		(end 130.873 59.623)
+		(start 131.1625 60.5)
+		(end 131.1625 59.9125)
 		(width 0.2)
 		(layer "F.Cu")
@@
 	)
 	(segment
-		(start 130.873 59.623)
-		(end 124.038536 59.623)
+		(start 121 61.377)
+		(end 120.541 61.836)
 		(width 0.2)
 		(layer "F.Cu")
@@
 	)
 	(segment
-		(start 124.038536 59.623)
-		(end 122.284536 61.377)
+		(start 130.873 59.623)
+		(end 124.038536 59.623)
 		(width 0.2)
 		(layer "F.Cu")
@@
 	)
 	(segment
-		(start 121.77 103.31)
-		(end 120.71 102.25)
+		(start 120.58 107.2)
+		(end 121.77 108.39)
 		(width 0.2)
 		(layer "F.Cu")
@@
 	)
 	(segment
-		(start 118.5 102.25)
-		(end 117.25 101)
+		(start 149.25 58.75)
+		(end 118 58.75)
 		(width 0.2)
 		(layer "F.Cu")
@@
 	(segment
 		(start 149.9125 59.4125)
-		(end 149.9125 60.5)
+		(end 149.25 58.75)
 		(width 0.2)
 		(layer "F.Cu")
@@
 	)
 	(segment
-		(start 149.25 58.75)
-		(end 149.9125 59.4125)
+		(start 118 58.75)
+		(end 117.25 59.5)
 		(width 0.2)
 		(layer "F.Cu")
@@
 	)
 	(segment
-		(start 117.25 101)
-		(end 117.25 59.5)
+		(start 117.25 59.5)
+		(end 117.25 106.35)
 		(width 0.2)
 		(layer "F.Cu")
@@
 	)
 	(segment
-		(start 118 58.75)
-		(end 149.25 58.75)
+		(start 149.9125 60.5)
+		(end 149.9125 59.4125)
 		(width 0.2)
 		(layer "F.Cu")
@@
 	)
 	(segment
-		(start 120.71 102.25)
-		(end 118.5 102.25)
+		(start 118.1 107.2)
+		(end 120.58 107.2)
 		(width 0.2)
 		(layer "F.Cu")
@@
 	)
 	(segment
-		(start 117.25 59.5)
-		(end 118 58.75)
+		(start 117.25 106.35)
+		(end 118.1 107.2)
 		(width 0.2)
 		(layer "F.Cu")
@@
 	)
 	(segment
-		(start 143.575 60.5)
-		(end 143.575 59.616)
+		(start 118.120536 59.041)
+		(end 117.541 59.620536)
 		(width 0.2)
 		(layer "F.Cu")
@@
 	)
 	(segment
-		(start 143 59.041)
-		(end 118.120536 59.041)
+		(start 117.541 59.620536)
+		(end 117.541 103.441)
 		(width 0.2)
 		(layer "F.Cu")
@@
 	)
 	(segment
-		(start 117.541 59.620536)
-		(end 117.541 98.541)
+		(start 117.541 103.441)
+		(end 118.8 104.7)
 		(width 0.2)
 		(layer "F.Cu")
@@
 	)
 	(segment
-		(start 120.5 99.5)
-		(end 121.77 100.77)
+		(start 143.575 59.616)
+		(end 143 59.041)
 		(width 0.2)
 		(layer "F.Cu")
@@
 	)
 	(segment
-		(start 118.5 99.5)
-		(end 120.5 99.5)
+		(start 118.8 104.7)
+		(end 120.62 104.7)
 		(width 0.2)
 		(layer "F.Cu")
@@
 	)
 	(segment
-		(start 143.575 59.616)
-		(end 143 59.041)
+		(start 143 59.041)
+		(end 118.120536 59.041)
 		(width 0.2)
 		(layer "F.Cu")
@@
 	)
 	(segment
-		(start 117.541 98.541)
-		(end 118.5 99.5)
+		(start 143.575 60.5)
+		(end 143.575 59.616)
 		(width 0.2)
 		(layer "F.Cu")
@@
 	)
 	(segment
-		(start 118.120536 59.041)
-		(end 117.541 59.620536)
+		(start 120.62 104.7)
+		(end 121.77 105.85)
 		(width 0.2)
 		(layer "F.Cu")
@@
 	(segment
 		(start 122.164 61.086)
-		(end 123.918 59.332)
+		(end 120.664 61.086)
 		(width 0.2)
 		(layer "F.Cu")
@@
 	)
 	(segment
-		(start 123.918 59.332)
-		(end 124.25 59.332)
+		(start 120.25 101.79)
+		(end 121.77 103.31)
 		(width 0.2)
 		(layer "F.Cu")
@@
 	)
 	(segment
-		(start 137.4125 59.7445)
-		(end 137 59.332)
+		(start 137 59.332)
+		(end 123.918 59.332)
 		(width 0.2)
 		(layer "F.Cu")
@@
 	)
 	(segment
-		(start 122 61.086)
+		(start 123.918 59.332)
 		(end 122.164 61.086)
 		(width 0.2)
@@
 	)
 	(segment
-		(start 120.25 61.5)
-		(end 120.664 61.086)
-		(width 0.2)
-		(layer "F.Cu")
-		(net 96)
-	)
-	(segment
-		(start 120.25 94.75)
-		(end 120.25 61.5)
-		(width 0.2)
-		(layer "F.Cu")
-		(net 96)
-	)
-	(segment
 		(start 137.4125 60.5)
 		(end 137.4125 59.7445)
@@
 	)
 	(segment
-		(start 124.25 59.332)
+		(start 137.4125 59.7445)
 		(end 137 59.332)
 		(width 0.2)
@@
 	(segment
 		(start 120.664 61.086)
-		(end 122 61.086)
-		(width 0.2)
-		(layer "F.Cu")
-		(net 96)
-	)
-	(segment
-		(start 121.77 98.23)
-		(end 120.25 96.71)
+		(end 120.25 61.5)
 		(width 0.2)
 		(layer "F.Cu")
@@
 	)
 	(segment
-		(start 120.25 96.71)
-		(end 120.25 94.75)
+		(start 120.25 61.5)
+		(end 120.25 101.79)
 		(width 0.2)
 		(layer "F.Cu")
