File: Hardware/CAN_UART/can.kicad_sch (KiCad schematic)
At the start: 14 parts, among them U1 ADM3057ExRW

Commit message: analog & can finished
Connections:
- net CAN.N renamed CAN_N
- net CAN.P renamed CAN_P
- net CAN.RX renamed CAN_RX
- net CAN.TX renamed CAN_TX
- net STBY_CAN: no longer names the net of U1.8 (STBY)
- no-connect marks 2 -> 3
Other:
- note added: "Isolation"
- moved on the sheet: C5, C6, C7, C8
