File: Hardware/Power/power_section.kicad_sch (KiCad schematic)
At the start: 48 parts, among them Q1 SI2347DS-T1-GE3, T1 10V, T2 VCC, T3 GND, T4 GND, T5 5V, T6 3V3, T7 GND, U1 TPS563200, U2 TPS563300DRLR, U3 LM1117-3.3

Commit message: schematic update & pcb update
Parts:
- removed C14: 100n, symbol Device:C_Small
- removed C16: 47u, symbol Device:C_Small
- removed D4: LD10V, LED_SMD:LED_0603_1608Metric_Pad1.05x0.95mm_HandSolder, symbol Device:LED_Small
- removed F4: Polyfuse_Small, symbol Device:Polyfuse_Small
- removed L2: 10u, symbol Device:L_Small
- removed R2: 10k, symbol Device:R
- removed R5, R8: 1k, Resistor_SMD:R_0603_1608Metric_Pad0.98x0.95mm_HandSolder, symbol Device:R_Small
- removed R6: 115k, symbol Device:R_Small
- removed R7: 10k, symbol Device:R_Small
- removed T1: 10V, TestPoint:TestPoint_Pad_1.0x1.0mm, symbol Connector:TestPoint_Small
- removed U2: TPS563300DRLR, Package_TO_SOT_SMD:SOT-583-8, symbol Regulator_Switching:TPS563300
- added PS1: DPUN02N-15, PLC_STM:DPUN02N15, symbol PLC_on_STM:DPUN02N-15
- added R2: 56k2, Resistor_SMD:R_0603_1608Metric_Pad0.98x0.95mm_HandSolder, symbol Device:R_Small
- added T2: 15V, TestPoint:TestPoint_Pad_1.0x1.0mm, symbol Connector:TestPoint_Small
- added T5: GND, TestPoint:TestPoint_Pad_1.0x1.0mm, symbol Connector:TestPoint_Small
- added T6: +15V, TestPoint:TestPoint_Pad_1.0x1.0mm, symbol Connector:TestPoint_Small
- added T7: -15V, TestPoint:TestPoint_Pad_1.0x1.0mm, symbol Connector:TestPoint_Small
- C1, C10, C2: footprint (none) -> Capacitor_SMD:C_0603_1608Metric_Pad1.08x0.95mm_HandSolder; Mouser Part Number (none) -> 81-GRM188R6YA106MA3J; Mouser Price/Stock (none) -> https://www.mouser.pl/ProductDetail/Murata-Electronics/GRM1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
- C11: value 100n -> 10u; footprint (none) -> Capacitor_SMD:C_0603_1608Metric_Pad1.08x0.95mm_HandSolder; Mouser Part Number (none) -> 81-GRM188R6YA106MA3J; Mouser Price/Stock (none) -> https://www.mouser.pl/ProductDetail/Murata-Electronics/GRM1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
- C5: footprint (none) -> Capacitor_SMD:C_0603_1608Metric_Pad1.08x0.95mm_HandSolder; Mouser Part Number (none) -> GRM033R6YA104ME14D; Mouser Price/Stock (none) -> https://www.mouser.pl/ProductDetail/Murata-Electronics/GRM0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
- C8, C9: footprint (none) -> Capacitor_SMD:C_0603_1608Metric_Pad1.08x0.95mm_HandSolder; Mouser Part Number (none) -> 810-C2012X5R1V226MAC; Mouser Price/Stock (none) -> https://www.mouser.pl/ProductDetail/TDK/C2012X5R1V226M125AC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
- D3: value LD10V -> LD5V
- F2: value Polyfuse_Small -> 6V/1A; footprint (none) -> Fuse:Fuse_0805_2012Metric_Pad1.15x1.40mm_HandSolder; Mouser Part Number (none) -> 650-PICOSMDC050S-2; Mouser Price/Stock (none) -> https://www.mouser.pl/ProductDetail/Littelfuse/PICOSMDC050S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
- L1: value 4u7 -> 3u3/4A95; footprint (none) -> Inductor_SMD:L_TDK_VLS6045EX_VLS6045AF; Mouser Part Number (none) -> 810-VLS6045EX-3R3N; Mouser Price/Stock (none) -> https://www.mouser.pl/ProductDetail/TDK/VLS6045EX-3R3N?qs=o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
- R3: value 54k9 -> 10k; footprint (none) -> Resistor_SMD:R_0603_1608Metric_Pad0.98x0.95mm_HandSolder; Mouser Part Number (none) -> 71-CRCW0603-10K-E3; Mouser Price/Stock (none) -> https://www.mouser.pl/ProductDetail/Vishay/CRCW060310K0FKEA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
- R4: value 10k -> 1k; footprint (none) -> Resistor_SMD:R_0603_1608Metric_Pad0.98x0.95mm_HandSolder; Mouser Part Number (none) -> 71-CRCW06031K00FKED; Mouser Price/Stock (none) -> https://www.mouser.pl/ProductDetail/Vishay-Dale/CRCW06031K0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
- T4: value GND -> 5V
- U1: Mouser Part Number (none) -> 595-TPS563200DDCR; Mouser Price/Stock (none) -> https://www.mouser.pl/ProductDetail/Texas-Instruments/TPS56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
- renumbered C15 to C14, C17 to C15, D5 to D4, R9 to R5, T2 to T1, T7 to T10, T5 to T8, T6 to T9, U3 to U2
Connections:
- net +10V is gone; now on net +15V: C1.1, C2.1, U1.3 (VIN)
- net +5V: now also F2.2; no longer F2.1
- net D5V_R1k: now also R4.2
- net GND: now also C11.1, R3.1, PS1.2 (-VIN), PS1.6 (COMMON), T5.1; no longer C11.2, R4.2, T4.1
- net VCC_IN: now also PS1.1 (+VIN); no longer C10.1, C11.1
- net at R3.2, U1.4 (VFB): now also R2.2; no longer R4.1
- net at C8.1, C9.1, L1.2: now also F2.1, R4.1, T4.1, R2.1; no longer F2.2, R3.1
- net +15V: now reaches U1.5 (EN)
- net +15V: now also C10.1, PS1.5 (-VOUT), T2.1, T6.1
- new net -15V: C11.2, PS1.7 (+VOUT), T7.1
- no-connect marks 1 -> 0
Other:
- note added: "Designed by WEBENCH - check documentation directory for more details"
- note added: "POWER +15V TO +5V"
- note added: "POWER +24V TO -+15V"
- note removed: "Designed by WEBENCH - check documentation directory for details"
- note removed: "POWER +10V TO +5V"
- note removed: "POWER +24V TO +10V"

Commit message: schematic update & pcb update
Connections:
- net +5V_OUT: now reaches C8.1, C9.1, F2.1, L1.2, R2.1, R4.1, T4.1
- net FB_+5V: now reaches R2.2, R3.2, U1.4 (VFB)
- net SW_+5V: now reaches C5.1, L1.1, U1.2 (SW)
- net VBST_+5V: now reaches C5.2, U1.6 (VBST)
Changed lines of the file:
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@@
 		)
 	)
+	(label "FB_+5V"
+		(at 90.17 133.35 0)
+		(effects
+			(font
+				(size 0.508 0.508)
+			)
+			(justify left bottom)
+		)
+	)
 	(label "RPP_D"
 		(at 57.15 58.42 180)
@@
 		)
 	)
+	(label "SW_+5V"
+		(at 90.17 128.27 0)
+		(effects
+			(font
+				(size 0.508 0.508)
+			)
+			(justify left bottom)
+		)
+	)
 	(label "VO_+3.3V"
 		(at 224.79 127 0)
@@
 		)
 	)
+	(label "+5V_OUT"
+		(at 114.3 128.27 0)
+		(effects
+			(font
+				(size 0.5 0.5)
+			)
+			(justify left bottom)
+		)
+	)
+	(label "VBST_+5V"
+		(at 90.17 130.81 0)
+		(effects
+			(font
+				(size 0.508 0.508)
+			)
+			(justify left bottom)
+		)
+	)
 	(symbol
 		(lib_id "Device:Polyfuse_Small")
@@
 		(on_board yes)
 		(dnp no)
-		(property "Reference" "#FLG03"
+		(property "Reference" "#FLG05"
 			(at 227.965 116.84 0)
 			(effects
@@
 			(project "power"
 				(path "/b652b05a-4e3d-4ad1-b032-18886abe7d45/41e43fed-5c1d-4ba4-a553-b31d87724d09"
-					(reference "#FLG03")
+					(reference "#FLG05")
 					(unit 1)
 				)
@@
 		(dnp no)
 		(fields_autoplaced yes)
-		(property "Reference" "#PWR02"
+		(property "Reference" "#PWR04"
 			(at 80.01 161.29 0)
 			(effects
@@
 			(project "power"
 				(path "/b652b05a-4e3d-4ad1-b032-18886abe7d45/41e43fed-5c1d-4ba4-a553-b31d87724d09"
-					(reference "#PWR02")
+					(reference "#PWR04")
 					(unit 1)
 				)
@@
 		(dnp no)
 		(fields_autoplaced yes)
-		(property "Reference" "#PWR022"
+		(property "Reference" "#PWR05"
 			(at 143.51 119.38 0)
 			(effects
@@
 			(project ""
 				(path "/b652b05a-4e3d-4ad1-b032-18886abe7d45/41e43fed-5c1d-4ba4-a553-b31d87724d09"
-					(reference "#PWR022")
+					(reference "#PWR05")
 					(unit 1)
 				)
@@
 		(dnp no)
 		(fields_autoplaced yes)
-		(property "Reference" "#FLG05"
+		(property "Reference" "#FLG04"
 			(at 186.055 77.47 0)
 			(effects
@@
 			(project "power"
 				(path "/b652b05a-4e3d-4ad1-b032-18886abe7d45/41e43fed-5c1d-4ba4-a553-b31d87724d09"
-					(reference "#FLG05")
+					(reference "#FLG04")
 					(unit 1)
 				)
@@
 		(dnp no)
 		(fields_autoplaced yes)
-		(property "Reference" "#FLG04"
+		(property "Reference" "#FLG03"
 			(at 186.055 49.53 0)
 			(effects
@@
 			(project "power"
 				(path "/b652b05a-4e3d-4ad1-b032-18886abe7d45/41e43fed-5c1d-4ba4-a553-b31d87724d09"
-					(reference "#FLG04")
+					(reference "#FLG03")
 					(unit 1)
 				)
@@
 		(dnp no)
 		(fields_autoplaced yes)
-		(property "Reference" "#PWR05"
+		(property "Reference" "#PWR02"
 			(at 38.1 88.9 0)
 			(effects
@@
 			(project ""
 				(path "/b652b05a-4e3d-4ad1-b032-18886abe7d45/41e43fed-5c1d-4ba4-a553-b31d87724d09"
-					(reference "#PWR05")
+					(reference "#PWR02")
 					(unit 1)
 				)

Commit message: digital output & power finished
Parts:
- renumbered C12 to C10, C13 to C11, C10 to C12, C11 to C13, T8 to T6, T6 to T7, T7 to T8
Connections:
- net VCC_IN is gone; now on net +24V: C3.1, C4.1, C6.1, C7.1, D2.1 (K), PS1.1 (+VIN), Q1.2 (S)
- net +24V: no longer F1.2
- new net VCC: F1.2
Other:
- moved on the sheet: C12, C13, C3, C4, C6, C7, D1, D2, F1, PS1, Q1, R1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

Commit message: small adjustments
Parts:
- C11, C14, C5: Mouser Part Number GRM033R6YA104ME14D -> 81-GRM33R6YA104ME14D
Changed lines of the file:
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@@
 			)
 		)
-		(property "Mouser Part Number" "GRM033R6YA104ME14D"
+		(property "Mouser Part Number" "81-GRM33R6YA104ME14D"
 			(at 204.47 133.35 0)
 			(effects
@@
 			)
 		)
-		(property "Mouser Part Number" "GRM033R6YA104ME14D"
+		(property "Mouser Part Number" "81-GRM33R6YA104ME14D"
 			(at 229.87 133.35 0)
 			(effects
@@
 			)
 		)
-		(property "Mouser Part Number" "GRM033R6YA104ME14D"
+		(property "Mouser Part Number" "81-GRM33R6YA104ME14D"
 			(at 100.33 133.35 0)
 			(effects
